File: resistive-testboard/devboardmodule.kicad_sch (KiCad schematic)
At the start: 1 part

Commit message: fixed pinouts for ws2811 and pmos
Connections:
- net S2/SIG_IN: now also U1.3 (G_OUT); no longer U1.2 (G_OUT)
- net S3/SIG_IN: now also U1.4 (B_OUT); no longer U1.3 (B_OUT)
Changed lines of the file:
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@@
 	(wire
 		(pts
-			(xy 99.06 107.95) (xy 113.03 107.95)
-		)
-		(stroke
-			(width 0)
-			(type default)
-		)
-	)
-	(wire
-		(pts
-			(xy 101.6 110.49) (xy 101.6 127)
+			(xy 101.6 113.03) (xy 101.6 127)
 		)
 		(stroke
@@
 	(wire
 		(pts
+			(xy 99.06 110.49) (xy 106.68 110.49)
+		)
+		(stroke
+			(width 0)
+			(type default)
+		)
+	)
+	(wire
+		(pts
 			(xy 104.14 105.41) (xy 99.06 105.41)
 		)
@@
 	(wire
 		(pts
-			(xy 109.22 111.76) (xy 113.03 111.76)
+			(xy 106.68 110.49) (xy 106.68 107.95)
 		)
 		(stroke
@@
 	(wire
 		(pts
-			(xy 101.6 110.49) (xy 99.06 110.49)
+			(xy 106.68 107.95) (xy 113.03 107.95)
+		)
+		(stroke
+			(width 0)
+			(type default)
+		)
+	)
+	(wire
+		(pts
+			(xy 109.22 111.76) (xy 113.03 111.76)
 		)
 		(stroke
@@
 		(pts
 			(xy 113.03 90.17) (xy 104.14 90.17)
+		)
+		(stroke
+			(width 0)
+			(type default)
+		)
+	)
+	(wire
+		(pts
+			(xy 99.06 113.03) (xy 101.6 113.03)
 		)
 		(stroke
@@
 		(in_pos_files yes)
 		(dnp no)
-		(fields_autoplaced yes)
 		(property "Reference" "U1"
 			(at 82.55 108.5849 0)
