File: resistive-testboard/touchelectrode.kicad_sch (KiCad schematic)
At the start: 5 parts, among them Q1 PMOS

Commit message: fixed pinouts for ws2811 and pmos
Connections:
- net SIG_IN: now also Q1.1 (G); no longer Q1.2 (G)
- net VREF: now also Q1.2 (S); no longer Q1.3 (S)
- net at E1.1 (E), R3.1: now also Q1.3 (D); no longer Q1.1 (D)
