File: resistive-testboard/resistive-testboard.kicad_sch (KiCad schematic)
At the start: 2 parts, among them J1 Conn_01x04_Pin

Commit message: added pcb?
Parts:
- J1: footprint Connector_PinHeader_1.00mm:PinHeader_1x04_P1.00mm_Vertical -> Connector_PinHeader_2.54mm:PinHeader_1x04_P2.54mm_Vertical
Changed lines of the file:
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@@
 			)
 		)
-		(property "Footprint" "Connector_PinHeader_1.00mm:PinHeader_1x04_P1.00mm_Vertical"
+		(property "Footprint" "Connector_PinHeader_2.54mm:PinHeader_1x04_P2.54mm_Vertical"
 			(at 54.61 77.47 0)
 			(hide yes)

Commit message: moved pulldown resistor lower, added more copies of symbol
Connections:
- net +5V: now also J1.2 (Pin_2); no longer J1.3 (Pin_3)
- net GND: now also J1.4 (Pin_4); no longer J1.2 (Pin_2)
- net RX: now also J1.3 (Pin_3); no longer J1.4 (Pin_4)
Other:
- added sheet M3 (DevBoardModule.kicad_sch)
- added sheet M4 (DevBoardModule.kicad_sch)
